File: Control Boards/debug_control_board/debug_control_board.kicad_pcb (KiCad board)
At the start: 2 copper layers, 38.1 x 37.1 mm, 14 parts, among them J1 Conn_01x05, J10 Conn_01x26, J2 Conn_01x05, J3 Conn_01x04, J4 Conn_01x04, J5 Conn_01x05, J6 Conn_01x05, J7 Conn_01x02, J8 Conn_01x03, J9 Conn_01x26

Commit message: Updated debug board to support 30 pin ribbon cable
Parts:
- added J11: Conn_01x30, Connector_FFC-FPC:Hirose_FH12-30S-0.5SH_1x30-1MP_P0.50mm_Horizontal, B.Cu at (120.4, 86.8)
- added J12: Conn_01x30, Connector_FFC-FPC:Hirose_FH12-30S-0.5SH_1x30-1MP_P0.50mm_Horizontal, F.Cu at (120.4, 88.8)
- J10: value Conn_01x26 -> Conn_01x02; footprint Connector_FFC-FPC:Hirose_FH12-26S-0.5SH_1x26-1MP_P0.50mm_Horizontal -> Connector_PinHeader_2.54mm:PinHeader_1x02_P2.54mm_Vertical
- J9: value Conn_01x26 -> Conn_01x03; footprint Connector_FFC-FPC:Hirose_FH12-26S-0.5SH_1x26-1MP_P0.50mm_Horizontal -> Connector_PinHeader_2.54mm:PinHeader_1x03_P2.54mm_Vertical; moved to F.Cu
- moved J10 23.9 mm to (135.4, 106.4), turned to 90 degrees
- moved J9 20.8 mm to (130.1, 106.2), turned to 270 degrees
- moved REF** 5.01 mm to (146.2, 107.9)
- moved REF** 5.00 mm to (116.3, 107.9)
Connections:
- J10 pad 1: +5V -> /BOOT_SWITCH
- J9 pad 1: +5V -> /MOUSE_X
- J9 pad 2: GND -> /MOUSE_Y
- J9 pad 3: +3V3 -> GND
Routing:
- net /BOOT_SWITCH: track 0.00 -> 55.7 mm, vias 0 -> 1
- net /MOUSE_Y: track 0.00 -> 43.2 mm, vias 0 -> 1
- net /MOUSE_X: track 0.00 -> 43.1 mm, vias 0 -> 1
- net GND: track 6.61 -> 16.2 mm
- net +5V: track 34.3 -> 39.2 mm, vias 4 -> 1
- net +3V3: track 81.7 -> 77.7 mm
Other:
- board size 38.1 x 37.1 mm -> 38.1 x 42.2 mm
