File: Full Keyboard V2.0/FullKeyboardV1.kicad_pcb (KiCad board)
At the start: 2 copper layers, 305.6 x 104.9 mm, 616 parts, among them J1 Conn_01x30, J2 USB_C_Receptacle_USB2.0, J3 USB_A, J4 USB_A, J5 USB_A, J6 Conn_01x04, P7 AMS1117, SW1 Esc, SW10 2, SW11 W, SW12 S, SW13 Z, SW15 3, SW16 E, SW17 D, SW18 X, SW19 4, SW2 Tab, SW20 R, SW21 F, SW22 C, SW23 5, SW24 T, SW25 G, SW26 V, SW27 6, SW28 Y, SW29 H, SW3 Caps, SW30 B, SW32 7, SW33 U, SW34 J, SW35 N, SW36 8, SW37 I, SW38 K, SW39 M, SW4 double_key, SW40 9, SW41 O, SW42 L, SW43 <, SW44 0, SW45 P, SW46 ;, SW47 >, SW49 Minus, SW5 End/Home, SW50 [, SW51 ", SW52 /, SW54 =, SW55 ], SW59 BKSPC, SW6 1, SW60 \, SW61 Enter, SW63 Til, SW64 Del, SW65 Pg Up, SW66 Pg Dw, SW7 Q, SW8 A, SW9 double_key, T1 Vin, T3 Vout, U1 AT24C02, U2 FE1.1s, U3 CD74HC4067SM, U5 Cherry_bottom_row, Y1 12MHz

Commit message: Added BOOT switch
Parts:
- added REF**411: Stitching-Via-0.6mm, keyboard:Stitching-Via-0.6mm, F.Cu at (209.3, 50.8)
- added SW14: SW_SPDT, keyboard:SS12F23, B.Cu at (122.0, 52.1)
Connections:
- J1 pad 29: Net-(J1-Pad29) -> /MicroSheet/BOOT_SWITCH
Routing:
- net /MicroSheet/MOUSE_X: track 371.8 -> 225.2 mm
- net /MicroSheet/BOOT_SWITCH: track 0.00 -> 93.4 mm, vias 0 -> 3
- net /MicroSheet/MOUSE_Y: track 269.9 -> 227.4 mm
- net GND: track 67.7 -> 58.0 mm, vias 11 -> 12
- net +5V: track 279.5 -> 287.1 mm
- net +3V3: track 2550.0 -> 2551.9 mm
- net Net-(U2-Pad3): track 17.9 -> 18.5 mm

Commit message: added hotswap sockets
Parts:
- removed the REF**411 at (202.2, 122.1)
- removed the REF**411 at (215.5, 100.9)
- removed the REF**421 at (214.5, 100.9)
- removed the REF**421 at (202.9, 121.4)
- removed the REF**422 at (252.0, 86.5)
- removed the REF**423 at (252.0, 87.5)
- removed the REF**431 at (213.5, 100.9)
- removed the REF**431 at (203.6, 120.7)
- removed the REF**431 at (66.9, 74.7)
- removed the REF**431 at (223.3, 71.7)
- removed the REF**432 at (67.9, 74.7)
- removed the REF**432 at (223.3, 70.7)
- removed the REF**433 at (68.9, 74.7)
- removed the REF**433 at (223.3, 69.7)
- added REF**31: Stitching-Via-0.6mm, keyboard:Stitching-Via-0.6mm, F.Cu at (224.5, 71.0)
- added REF**411: Stitching-Via-0.6mm, keyboard:Stitching-Via-0.6mm, F.Cu at (218.0, 105.2)
- added REF**421: Stitching-Via-0.6mm, keyboard:Stitching-Via-0.6mm, F.Cu at (218.0, 106.2)
- added REF**431: Stitching-Via-0.6mm, keyboard:Stitching-Via-0.6mm, F.Cu at (22.5, 88.8)
- added REF**431: Stitching-Via-0.6mm, keyboard:Stitching-Via-0.6mm, F.Cu at (218.0, 107.2)
- added REF**431: Stitching-Via-0.6mm, keyboard:Stitching-Via-0.6mm, F.Cu at (42.2, 89.7)
- added REF**431: Stitching-Via-0.6mm, keyboard:Stitching-Via-0.6mm, F.Cu at (61.2, 89.6)
- added REF**431: Stitching-Via-0.6mm, keyboard:Stitching-Via-0.6mm, F.Cu at (118.3, 89.1)
- added REF**431: Stitching-Via-0.6mm, keyboard:Stitching-Via-0.6mm, F.Cu at (156.2, 88.8)
- added REF**431: Stitching-Via-0.6mm, keyboard:Stitching-Via-0.6mm, F.Cu at (194.3, 88.9)
- added REF**432: Stitching-Via-0.6mm, keyboard:Stitching-Via-0.6mm, F.Cu at (22.5, 87.8)
- added REF**432: Stitching-Via-0.6mm, keyboard:Stitching-Via-0.6mm, F.Cu at (42.2, 88.7)
- added REF**432: Stitching-Via-0.6mm, keyboard:Stitching-Via-0.6mm, F.Cu at (61.2, 88.6)
- added REF**432: Stitching-Via-0.6mm, keyboard:Stitching-Via-0.6mm, F.Cu at (118.3, 88.1)
- added REF**432: Stitching-Via-0.6mm, keyboard:Stitching-Via-0.6mm, F.Cu at (156.2, 87.8)
- added REF**432: Stitching-Via-0.6mm, keyboard:Stitching-Via-0.6mm, F.Cu at (194.3, 87.9)
- added REF**433: Stitching-Via-0.6mm, keyboard:Stitching-Via-0.6mm, F.Cu at (22.5, 86.8)
- added REF**433: Stitching-Via-0.6mm, keyboard:Stitching-Via-0.6mm, F.Cu at (42.2, 87.7)
- added REF**433: Stitching-Via-0.6mm, keyboard:Stitching-Via-0.6mm, F.Cu at (61.2, 87.6)
- added REF**433: Stitching-Via-0.6mm, keyboard:Stitching-Via-0.6mm, F.Cu at (118.3, 87.1)
- added REF**433: Stitching-Via-0.6mm, keyboard:Stitching-Via-0.6mm, F.Cu at (156.2, 86.8)
- added REF**433: Stitching-Via-0.6mm, keyboard:Stitching-Via-0.6mm, F.Cu at (194.3, 86.9)
- SW1, SW10, SW11, SW12, SW13, SW15, SW16, SW17, SW18, SW19, SW20, SW21, SW22, SW23, SW24, SW25, SW26, SW27, SW28, SW29, SW30, SW32, SW33, SW34, SW35, SW36, SW37, SW38, SW39, SW40, SW41, SW42, SW43, SW44, SW45, SW46, SW47, SW49, SW5, SW50, SW51, SW52, SW54, SW55, SW6, SW63, SW64, SW65, SW66, SW7, SW8: footprint keyboard:RGB_CHERRY_PCB_100H -> keyboard:RGB_CHERRY_PCB_100H_HOTSWAP
- SW2, SW60: footprint keyboard:RGB_CHERRY_PCB_150H -> keyboard:RGB_CHERRY_PCB_150H_HOTSWAP
- SW3: footprint keyboard:RGB_CHERRY_PCB_175H -> keyboard:RGB_CHERRY_PCB_175H_HOTSWAP
- SW61: footprint keyboard:RGB_CHERRY_PCB_225H -> keyboard:RGB_CHERRY_PCB_225H_HOTSWAP
- moved G*** 192.5 mm to (152.8, -89.7)
- moved G*** 189.1 mm to (129.5, -91.6)
- moved G*** 150.2 mm to (56.8, -27.3)
- moved G*** 150.2 mm to (57.1, -27.3)
- moved REF**41 59.0 mm to (224.5, 72.0), turned to 270 degrees
- moved REF**412 21.8 mm to (249.9, 108.2)
- moved REF**413 21.8 mm to (249.9, 109.2)
- moved D19 10.5 mm to (70.6, 73.9), turned to 270 degrees
- moved D4 10.4 mm to (-0.64, 117.1), turned to 90 degrees
- moved D6 10.1 mm to (12.6, 73.4), turned to 270 degrees
- moved D23 9.91 mm to (89.3, 73.3), turned to 270 degrees
- moved D27 9.89 mm to (108.1, 73.4), turned to 270 degrees
- moved D54 9.75 mm to (223.0, 72.3), turned to 270 degrees
- moved D15 9.45 mm to (51.0, 72.8), turned to 270 degrees
- moved D10 9.26 mm to (32.8, 72.8), turned to 270 degrees
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Routing:
- net /ROW1: track 316.1 -> 372.4 mm
- net /ROW2: track 413.5 -> 466.7 mm
- net /COL14: track 242.5 -> 190.0 mm
- net /ROW0: track 318.8 -> 369.8 mm
- net /ROW3: track 377.5 -> 421.5 mm
- net GND: track 58.0 -> 45.5 mm, vias 12 -> 11
- net Net-(D64-Pad1): track 2.44 -> 14.8 mm
- net Net-(D65-Pad1): track 2.48 -> 13.4 mm
- net Net-(D66-Pad1): track 2.49 -> 13.1 mm
- net Net-(D68-Pad1): track 4.09 -> 14.4 mm
- net +3V3: track 2551.9 -> 2562.1 mm, vias 81 -> 80
- net Net-(D6-Pad1): track 4.15 -> 13.1 mm
- net Net-(D27-Pad1): track 4.99 -> 13.6 mm
- net /COL6: track 193.6 -> 185.1 mm
- net Net-(D23-Pad1): track 5.47 -> 14.0 mm
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
Commit message: Modified mounting holes
Parts:
- removed REF** (x8): 1pin, Connect:1pin
- added REF**431: Stitching-Via-0.6mm, keyboard:Stitching-Via-0.6mm, F.Cu at (291.9, 83.7)
- added REF**432: Stitching-Via-0.6mm, keyboard:Stitching-Via-0.6mm, F.Cu at (292.9, 83.7)
- added REF**433: Stitching-Via-0.6mm, keyboard:Stitching-Via-0.6mm, F.Cu at (293.9, 83.7)
- moved REF**411 7.68 mm to (17.4, 141.9)
- moved REF**412 7.68 mm to (17.4, 142.9)
- moved REF**421 7.68 mm to (18.4, 141.9)
- moved REF**422 7.68 mm to (18.4, 142.9)
- moved REF**431 7.68 mm to (19.4, 141.9)
- moved REF**432 7.68 mm to (19.4, 142.9)
- moved REF**41 1.40 mm to (292.4, 91.9)
- moved C24 1.39 mm to (281.9, 146.2), turned to 315 degrees
Routing:
- net +3V3: track 2562.1 -> 2569.3 mm
- net /RGB4: track 466.9 -> 469.7 mm
- net /RGB3: track 438.4 -> 441.0 mm
- net /COL0: track 294.8 -> 295.4 mm
Other:
- outline, holes or cut-outs redrawn
