File: Test Pad/Keypad/PowerSchematic.kicad_sch (KiCad schematic)
At the start: 10 parts

Commit message: Started nucleo 144 test pad and keypad boards
Parts:
- C66: value (none) -> C; footprint (none) -> Capacitor_SMD:C_0603_1608Metric
- C67: value (none) -> CP1; footprint (none) -> Capacitor_SMD:C_0603_1608Metric
- J2: value (none) -> USB_C_Receptacle_USB2.0; footprint (none) -> Connector_USB:USB_C_Receptacle_HRO_TYPE-C-31-M-12
- P7: value (none) -> AMS1117; footprint (none) -> Package_TO_SOT_SMD:SOT-223
- R11, R12: value (none) -> 5K1; footprint (none) -> Resistor_SMD:R_0603_1608Metric
- R6, R7: value (none) -> R; footprint (none) -> Resistor_SMD:R_0603_1608Metric
- T1: value (none) -> Vin; footprint (none) -> TestPoint:TestPoint_Pad_1.0x1.0mm
- T3: value (none) -> Vout; footprint (none) -> TestPoint:TestPoint_Pad_1.0x1.0mm
Changed lines of the file:
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@@
       (effects (font (size 1.524 1.524)))
     )
-    (property "Value" "" (id 1) (at 123.19 69.85 0)
-      (effects (font (size 1.524 1.524)))
-    )
-    (property "Footprint" "" (id 2) (at 123.19 74.93 0)
+    (property "Value" "Vin" (id 1) (at 123.19 69.85 0)
+      (effects (font (size 1.524 1.524)))
+    )
+    (property "Footprint" "TestPoint:TestPoint_Pad_1.0x1.0mm" (id 2) (at 123.19 74.93 0)
       (effects (font (size 1.524 1.524)) hide)
     )
@@
       (effects (font (size 1.27 1.27)) hide)
     )
-    (property "Value" "" (id 1) (at 94.615 116.84 0))
+    (property "Value" "GND" (id 1) (at 94.615 116.84 0))
     (property "Footprint" "" (id 2) (at 94.615 113.03 0))
     (property "Datasheet" "" (id 3) (at 94.615 113.03 0))
@@
       (effects (font (size 1.524 1.524)))
     )
-    (property "Value" "" (id 1) (at 141.605 69.215 0)
-      (effects (font (size 1.524 1.524)))
-    )
-    (property "Footprint" "" (id 2) (at 138.43 74.93 0)
+    (property "Value" "AMS1117" (id 1) (at 141.605 69.215 0)
+      (effects (font (size 1.524 1.524)))
+    )
+    (property "Footprint" "Package_TO_SOT_SMD:SOT-223" (id 2) (at 138.43 74.93 0)
       (effects (font (size 1.524 1.524)) hide)
     )
@@
     (in_bom yes) (on_board yes)
     (property "Reference" "R6" (id 0) (at 151.892 78.74 90))
-    (property "Value" "" (id 1) (at 149.86 78.74 90))
-    (property "Footprint" "" (id 2) (at 148.082 78.74 90)
+    (property "Value" "R" (id 1) (at 149.86 78.74 90))
+    (property "Footprint" "Resistor_SMD:R_0603_1608Metric" (id 2) (at 148.082 78.74 90)
       (effects (font (size 1.27 1.27)) hide)
     )
@@
     (in_bom yes) (on_board yes)
     (property "Reference" "R7" (id 0) (at 151.892 86.36 90))
-    (property "Value" "" (id 1) (at 149.86 86.36 90))
-    (property "Footprint" "" (id 2) (at 148.082 86.36 90)
+    (property "Value" "R" (id 1) (at 149.86 86.36 90))
+    (property "Footprint" "Resistor_SMD:R_0603_1608Metric" (id 2) (at 148.082 86.36 90)
       (effects (font (size 1.27 1.27)) hide)
     )
@@
       (effects (font (size 1.27 1.27)) hide)
     )
-    (property "Value" "" (id 1) (at 149.86 92.71 0))
+    (property "Value" "GND" (id 1) (at 149.86 92.71 0))
     (property "Footprint" "" (id 2) (at 149.86 88.9 0))
     (property "Datasheet" "" (id 3) (at 149.86 88.9 0))
@@
       (effects (font (size 1.27 1.27)) (justify left))
     )
-    (property "Value" "" (id 1) (at 156.845 83.82 0)
-      (effects (font (size 1.27 1.27)) (justify left))
-    )
-    (property "Footprint" "" (id 2) (at 156.21 81.28 0)
+    (property "Value" "CP1" (id 1) (at 156.845 83.82 0)
+      (effects (font (size 1.27 1.27)) (justify left))
+    )
+    (property "Footprint" "Capacitor_SMD:C_0603_1608Metric" (id 2) (at 156.21 81.28 0)
       (effects (font (size 1.27 1.27)) hide)
     )
@@
       (effects (font (size 1.27 1.27)) hide)
     )
-    (property "Value" "" (id 1) (at 156.21 87.63 0))
+    (property "Value" "GND" (id 1) (at 156.21 87.63 0))
     (property "Footprint" "" (id 2) (at 156.21 83.82 0))
     (property "Datasheet" "" (id 3) (at 156.21 83.82 0))
@@
       (effects (font (size 1.27 1.27)) (justify left))
     )
-    (property "Value" "" (id 1) (at 127.635 83.82 0)
-      (effects (font (size 1.27 1.27)) (justify left))
-    )
-    (property "Footprint" "" (id 2) (at 127.9652 85.09 0)
+    (property "Value" "C" (id 1) (at 127.635 83.82 0)
+      (effects (font (size 1.27 1.27)) (justify left))
+    )
+    (property "Footprint" "Capacitor_SMD:C_0603_1608Metric" (id 2) (at 127.9652 85.09 0)
       (effects (font (size 1.27 1.27)) hide)
     )
@@
       (effects (font (size 1.27 1.27)) hide)
     )
-    (property "Value" "" (id 1) (at 127 87.63 0))
+    (property "Value" "GND" (id 1) (at 127 87.63 0))
     (property "Footprint" "" (id 2) (at 127 83.82 0))
     (property "Datasheet" "" (id 3) (at 127 83.82 0))
@@
       (effects (font (size 1.524 1.524)))
     )
-    (property "Value" "" (id 1) (at 163.83 67.31 0)
-      (effects (font (size 1.524 1.524)))
-    )
-    (property "Footprint" "" (id 2) (at 163.83 72.39 0)
+    (property "Value" "Vout" (id 1) (at 163.83 67.31 0)
+      (effects (font (size 1.524 1.524)))
+    )
+    (property "Footprint" "TestPoint:TestPoint_Pad_1.0x1.0mm" (id 2) (at 163.83 72.39 0)
       (effects (font (size 1.524 1.524)) hide)
     )
@@
       (effects (font (size 1.27 1.27)) hide)
     )
-    (property "Value" "" (id 1) (at 171.196 74.93 0))
+    (property "Value" "+3V3" (id 1) (at 171.196 74.93 0))
     (property "Footprint" "" (id 2) (at 167.64 74.93 0))
     (property "Datasheet" "" (id 3) (at 167.64 74.93 0))
@@
     (in_bom yes) (on_board yes)
     (property "Reference" "J2" (id 0) (at 97.3328 68.1482 0))
-    (property "Value" "" (id 1) (at 97.3328 70.4596 0))
-    (property "Footprint" "" (id 2) (at 98.425 90.17 0)
+    (property "Value" "USB_C_Receptacle_USB2.0" (id 1) (at 97.3328 70.4596 0))
+    (property "Footprint" "Connector_USB:USB_C_Receptacle_HRO_TYPE-C-31-M-12" (id 2) (at 98.425 90.17 0)
       (effects (font (size 1.27 1.27)) hide)
     )
@@
     (in_bom yes) (on_board yes)
     (property "Reference" "R11" (id 0) (at 112.395 78.105 90))
-    (property "Value" "" (id 1) (at 112.395 80.01 90))
-    (property "Footprint" "" (id 2) (at 112.395 78.232 90)
+    (property "Value" "5K1" (id 1) (at 112.395 80.01 90))
+    (property "Footprint" "Resistor_SMD:R_0603_1608Metric" (id 2) (at 112.395 78.232 90)
       (effects (font (size 1.27 1.27)) hide)
     )
@@
     (in_bom yes) (on_board yes)
     (property "Reference" "R12" (id 0) (at 112.395 84.582 90))
-    (property "Value" "" (id 1) (at 112.395 82.55 90))
-    (property "Footprint" "" (id 2) (at 112.395 80.772 90)
+    (property "Value" "5K1" (id 1) (at 112.395 82.55 90))
+    (property "Footprint" "Resistor_SMD:R_0603_1608Metric" (id 2) (at 112.395 80.772 90)
       (effects (font (size 1.27 1.27)) hide)
     )
@@
       (effects (font (size 1.27 1.27)) hide)
     )
-    (property "Value" "" (id 1) (at 118.745 80.01 0))
+    (property "Value" "GND" (id 1) (at 118.745 80.01 0))
     (property "Footprint" "" (id 2) (at 114.935 80.01 0))
     (property "Datasheet" "" (id 3) (at 114.935 80.01 0))
@@
       (effects (font (size 1.27 1.27)) hide)
     )
-    (property "Value" "" (id 1) (at 115.316 70.5358 0))
+    (property "Value" "+5V" (id 1) (at 115.316 70.5358 0))
     (property "Footprint" "" (id 2) (at 114.935 74.93 0)
       (effects (font (size 1.27 1.27)) hide)
